File: filaSens.brd (EAGLE design)
At the start: 50 x 20 mm, 16 parts, among them IC2 SS495, IC3 TINY85

Commit message: Add files via upload
Parts:
- moved R1 2.16 mm to (9.91, 6.35)
- moved C1 1.27 mm to (22.2, 6.35), turned to 270 degrees
- moved C2 1.27 mm to (21.0, 6.35), turned to 270 degrees
- moved LED1 1.27 mm to (11.4, 6.35), turned to 90 degrees
- turned R5 to 270 degrees
Routing:
- net +5V: track 66.6 -> 55.5 mm
- net GND: track 107.4 -> 104.7 mm, vias 6 -> 5
- net N$1: track 19.9 -> 22.4 mm
- net SDA: track 41.0 -> 43.1 mm
- net FAULT: track 47.7 -> 46.0 mm
- net MISO: track 35.9 -> 37.5 mm
- net N$2: track 2.60 -> 1.63 mm
- net IN: track 33.9 -> 34.6 mm
- net SCK: track 40.6 -> 41.3 mm
- net OUT: track 29.5 -> 28.9 mm
Other:
- board text added: "rev1A"
- board text removed: "rev1"

Commit message: Add files via upload
Parts:
- moved C1 0.13 mm to (22.2, 6.22)
- moved C2 0.13 mm to (21.0, 6.22)
Routing:
- net GND: track 104.7 -> 104.8 mm, vias 5 -> 3
Changed lines of the file:
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@@
 <attribute name="VALUE" x="28.194" y="8.255" size="1.27" layer="27" rot="R90"/>
 </element>
-<element name="C1" library="rcl" library_urn="urn:adsk.eagle:library:334" package="C0402" package3d_urn="urn:adsk.eagle:package:23626/2" value="10uF" x="22.225" y="6.35" smashed="yes" rot="R270" grouprefs="ACTIVE">
+<element name="C1" library="rcl" library_urn="urn:adsk.eagle:library:334" package="C0402" package3d_urn="urn:adsk.eagle:package:23626/2" value="10uF" x="22.225" y="6.223" smashed="yes" rot="R270" grouprefs="ACTIVE">
 <attribute name="NAME" x="21.59" y="4.445" size="1.27" layer="25" rot="R270"/>
-<attribute name="POPULARITY" value="18" x="22.225" y="6.35" size="1.778" layer="27" rot="R270" display="off"/>
-<attribute name="SPICEPREFIX" value="C" x="22.225" y="6.35" size="1.778" layer="27" rot="R270" display="off"/>
-<attribute name="VALUE" x="22.86" y="8.255" size="1.27" layer="27" rot="R90"/>
+<attribute name="POPULARITY" value="18" x="22.225" y="6.223" size="1.778" layer="27" rot="R270" display="off"/>
+<attribute name="SPICEPREFIX" value="C" x="22.225" y="6.223" size="1.778" layer="27" rot="R270" display="off"/>
+<attribute name="VALUE" x="22.86" y="8.128" size="1.27" layer="27" rot="R90"/>
 </element>
-<element name="C2" library="rcl" library_urn="urn:adsk.eagle:library:334" package="C0402" package3d_urn="urn:adsk.eagle:package:23626/2" value="10uF" x="20.955" y="6.35" smashed="yes" rot="R270" grouprefs="ACTIVE">
+<element name="C2" library="rcl" library_urn="urn:adsk.eagle:library:334" package="C0402" package3d_urn="urn:adsk.eagle:package:23626/2" value="10uF" x="20.955" y="6.223" smashed="yes" rot="R270" grouprefs="ACTIVE">
 <attribute name="NAME" x="20.32" y="4.445" size="1.27" layer="25" rot="R270"/>
-<attribute name="POPULARITY" value="18" x="20.955" y="6.35" size="1.778" layer="27" rot="R270" display="off"/>
-<attribute name="SPICEPREFIX" value="C" x="20.955" y="6.35" size="1.778" layer="27" rot="R270" display="off"/>
-<attribute name="VALUE" x="21.59" y="8.255" size="1.27" layer="27" rot="R90"/>
+<attribute name="POPULARITY" value="18" x="20.955" y="6.223" size="1.778" layer="27" rot="R270" display="off"/>
+<attribute name="SPICEPREFIX" value="C" x="20.955" y="6.223" size="1.778" layer="27" rot="R270" display="off"/>
+<attribute name="VALUE" x="21.59" y="8.128" size="1.27" layer="27" rot="R90"/>
 </element>
 <element name="S1" library="SparkFun-Switches" library_urn="urn:adsk.eagle:library:535" package="TACTILE_SWITCH_SMD_6.2MM_TALL" package3d_urn="urn:adsk.eagle:package:40172/1" value="MOMENTARY-SWITCH-SPST-SMD-6.2MM-TALL" x="4.445" y="6.35" smashed="yes" rot="R90">
@@
 <wire x1="24.765" y1="6.985" x2="24.765" y2="6.85" width="0.254" layer="1"/>
 <wire x1="23.495" y1="6.985" x2="22.225" y2="6.985" width="0.254" layer="1"/>
-<wire x1="22.225" y1="6.985" x2="22.225" y2="7" width="0.254" layer="1"/>
+<wire x1="22.225" y1="6.985" x2="22.225" y2="6.873" width="0.254" layer="1"/>
 <wire x1="23.495" y1="6.985" x2="23.495" y2="6.85" width="0.254" layer="1"/>
 <wire x1="26.67" y1="4.445" x2="26.035" y2="5.08" width="0.254" layer="1"/>
@@
 <wire x1="45.72" y1="16.51" x2="45.72" y2="16.375" width="0.254" layer="1"/>
 <wire x1="40.64" y1="16.51" x2="40.64" y2="16.375" width="0.254" layer="1"/>
-<wire x1="18.415" y1="5.969" x2="19.939" y2="7.493" width="0.254" layer="1"/>
-<wire x1="18.415" y1="3.4925" x2="18.415" y2="5.969" width="0.254" layer="1"/>
+<wire x1="19.939" y1="7.493" x2="18.415" y2="5.969" width="0.254" layer="1"/>
 <wire x1="19.939" y1="14.6685" x2="17.78" y2="16.8275" width="0.254" layer="1"/>
 <wire x1="19.939" y1="7.493" x2="19.939" y2="9.271" width="0.254" layer="1"/>
@@
 <wire x1="25.4" y1="8.255" x2="20.955" y2="8.255" width="0.254" layer="1"/>
 <wire x1="19.939" y1="9.271" x2="20.955" y2="8.255" width="0.254" layer="1"/>
-<wire x1="20.955" y1="8.255" x2="20.955" y2="7" width="0.254" layer="1"/>
+<wire x1="20.955" y1="8.255" x2="20.955" y2="6.873" width="0.254" layer="1"/>
+<wire x1="18.415" y1="5.969" x2="18.415" y2="4.064" width="0.254" layer="1"/>
+<wire x1="18.415" y1="4.064" x2="18.415" y2="3.4925" width="0" layer="19" extent="1-1"/>
 </signal>
 <signal name="GND" class="1">
@@
 <wire x1="16.51" y1="14.605" x2="16.51" y2="17.01" width="0.254" layer="1"/>
 <wire x1="8.89" y1="13.335" x2="15.24" y2="13.335" width="0.254" layer="1"/>
-<wire x1="14.605" y1="5.715" x2="19.685" y2="5.715" width="0.254" layer="16"/>
-<wire x1="14.605" y1="5.715" x2="11.43" y2="8.89" width="0.254" layer="16"/>
 <wire x1="11.43" y1="8.89" x2="11.43" y2="18.415" width="0.254" layer="16"/>
 <wire x1="11.43" y1="18.415" x2="11.811" y2="18.796" width="0.254" layer="16"/>
 <wire x1="11.811" y1="18.796" x2="16.51" y2="18.796" width="0.254" layer="16"/>
 <wire x1="16.51" y1="18.796" x2="16.51" y2="17.01" width="0.254" layer="16"/>
-<wire x1="19.7" y1="5.73" x2="19.685" y2="5.715" width="0.254" layer="1"/>
-<via x="19.685" y="5.715" extent="1-16" drill="0.35"/>
-<via x="19.685" y="5.715" extent="1-16" drill="0.35"/>
-<via x="19.685" y="5.715" extent="1-16" drill="0.35"/>
 <wire x1="24.765" y1="3.81" x2="26.035" y2="2.54" width="0.254" layer="1"/>
 <wire x1="24.765" y1="5.85" x2="24.765" y2="4.445" width="0.254" layer="1"/>
 <wire x1="24.765" y1="4.445" x2="24.765" y2="3.81" width="0.254" layer="1"/>
-<wire x1="19.685" y1="5.715" x2="20.955" y2="4.445" width="0.254" layer="16"/>
-<wire x1="20.955" y1="4.445" x2="24.765" y2="4.445" width="0.254" layer="16"/>
 <via x="24.765" y="4.445" extent="1-16" drill="0.35"/>
-<wire x1="19.685" y1="5.715" x2="20.94" y2="5.715" width="0.254" layer="1"/>
-<wire x1="20.94" y1="5.715" x2="20.955" y2="5.7" width="0.254" layer="1"/>
-<wire x1="20.955" y1="5.7" x2="22.225" y2="5.7" width="0.254" layer="1"/>
 <wire x1="4.445" y1="6.35" x2="5.08" y2="6.985" width="0.254" layer="1"/>
 <wire x1="11.313" y1="9.504" x2="9.906" y2="8.097" width="0.254" layer="1"/>
 <wire x1="9.906" y1="8.097" x2="9.906" y2="6.985" width="0.254" layer="1"/>
 <wire x1="14.615" y1="9.504" x2="11.313" y2="9.504" width="0.254" layer="1"/>
+<wire x1="20.955" y1="5.573" x2="20.925" y2="5.603" width="0.254" layer="1"/>
+<wire x1="22.225" y1="5.573" x2="20.955" y2="5.573" width="0.254" layer="1"/>
+<wire x1="24.765" y1="4.445" x2="20.701" y2="4.445" width="0.254" layer="16"/>
+<wire x1="19.558" y1="5.588" x2="19.573" y2="5.573" width="0.254" layer="1"/>
+<wire x1="20.955" y1="5.573" x2="19.573" y2="5.573" width="0.254" layer="1"/>
+<via x="19.558" y="5.588" extent="1-16" drill="0.35"/>
+<wire x1="19.558" y1="5.588" x2="14.732" y2="5.588" width="0.254" layer="16"/>
+<wire x1="14.732" y1="5.588" x2="11.43" y2="8.89" width="0.254" layer="16"/>
+<wire x1="19.558" y1="5.588" x2="20.701" y2="4.445" width="0.254" layer="16"/>
 </signal>
 <signal name="SDA">
